File: DIPduino.kicad_sch (KiCad schematic)
At the start: 39 parts, among them J1 USB_B, J10 3.3V Rail, J11 GND Rail, J2 BARREL JACK, J3 AVR ICSP, J4 5V Rail, J5 PIC ICSP, J6 Analog Pins, J7 Digital Pins 0-7, J8 Power Pins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

Commit message: added 7805 reg, R3
Parts:
- removed C8: 2.2uF, Capacitor_THT:C_Disc_D3.0mm_W1.6mm_P2.50mm, symbol Device:C
- removed U3: MIC2954, Package_TO_SOT_THT:TO-92_Inline, symbol Regulator_Linear:AP7384-33V
- added C8: 2.2 uf, Capacitor_THT:C_Disc_D3.0mm_W1.6mm_P2.50mm, symbol Device:C_Polarized
- added U4: L7805, Package_TO_SOT_THT:TO-220-3_Horizontal_TabDown, symbol Regulator_Linear:L7805
- U1: value ATmega328P-PU -> ATMEGA328P-PU
Connections:
- net +5V: now also C8.1, U4.3 (OUT)
- net GND: now also C8.2, U4.2 (GND)
- net VIN: now also U4.1 (IN)
Changed lines of the file:
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@@
     (effects (font (size 1.27 1.27)) (justify left bottom))
-  )
-  (symbol (lib_id "Regulator_Linear:AP7384-33V") (at 198.12 137.16 0) (unit 1)
-    (in_bom yes) (on_board yes) (dnp no)
-    (property "Reference" "U3" (at 198.12 130.81 0)
-      (effects (font (size 1.27 1.27)))
-    )
-    (property "Value" "MIC2954" (at 198.12 133.35 0)
-      (effects (font (size 1.27 1.27)))
-    )
-    (property "Footprint" "Package_TO_SOT_THT:TO-92_Inline" (at 196.85 127 0)
-      (effects (font (size 1.27 1.27) italic) hide)
-    )
-    (property "Datasheet" "https://www.diodes.com/assets/Datasheets/AP7384.pdf" (at 199.39 156.21 0)
-      (effects (font (size 1.27 1.27)) hide)
-    )
-    (pin "1")
-    (pin "2")
-    (pin "3")
-    (instances
-      (project "DIPduino"
-        (path "/2b19a4dd-043a-4133-8ff3-f6499add1fd2"
-          (reference "U3") (unit 1)
-        )
-      )
-    )
   )
   (symbol (lib_id "power:GND") (at 101.6 156.21 0) (unit 1)
@@
         (path "/2b19a4dd-043a-4133-8ff3-f6499add1fd2"
           (reference "#PWR010") (unit 1)
+        )
+      )
+    )
+  )
+  (symbol (lib_id "Regulator_Linear:L7805") (at 198.12 137.16 0) (unit 1)
+    (in_bom yes) (on_board yes) (dnp no) (fields_autoplaced)
+    (property "Reference" "U4" (at 198.12 130.81 0)
+      (effects (font (size 1.27 1.27)))
+    )
+    (property "Value" "L7805" (at 198.12 133.35 0)
+      (effects (font (size 1.27 1.27)))
+    )
+    (property "Footprint" "Package_TO_SOT_THT:TO-220-3_Horizontal_TabDown" (at 198.755 140.97 0)
+      (effects (font (size 1.27 1.27) italic) (justify left) hide)
+    )
+    (property "Datasheet" "http://www.st.com/content/ccc/resource/technical/document/datasheet/41/4f/b3/b0/12/d4/47/88/CD00000444.pdf/files/CD00000444.pdf/jcr:content/translations/en.CD00000444.pdf" (at 198.12 138.43 0)
+      (effects (font (size 1.27 1.27)) hide)
+    )
+    (pin "1")
+    (pin "2")
+    (pin "3")
+    (instances
+      (project "DIPduino"
+        (path "/2b19a4dd-043a-4133-8ff3-f6499add1fd2"
+          (reference "U4") (unit 1)
         )
       )
@@
         (path "/2b19a4dd-043a-4133-8ff3-f6499add1fd2"
           (reference "D1") (unit 1)
+        )
+      )
+    )
+  )
+  (symbol (lib_id "Device:C_Polarized") (at 224.79 143.51 0) (unit 1)
+    (in_bom yes) (on_board yes) (dnp no) (fields_autoplaced)
+    (property "Reference" "C8" (at 228.6 141.986 0)
+      (effects (font (size 1.27 1.27)) (justify left))
+    )
+    (property "Value" "2.2 uf" (at 228.6 144.526 0)
+      (effects (font (size 1.27 1.27)) (justify left))
+    )
+    (property "Footprint" "Capacitor_THT:C_Disc_D3.0mm_W1.6mm_P2.50mm" (at 225.7552 147.32 0)
+      (effects (font (size 1.27 1.27)) hide)
+    )
+    (property "Datasheet" "~" (at 224.79 143.51 0)
+      (effects (font (size 1.27 1.27)) hide)
+    )
+    (pin "1")
+    (pin "2")
+    (instances
+      (project "DIPduino"
+        (path "/2b19a4dd-043a-4133-8ff3-f6499add1fd2"
+          (reference "C8") (unit 1)
         )
       )
@@
     )
   )
-  (symbol (lib_id "Device:C") (at 224.79 143.51 0) (unit 1)
-    (in_bom yes) (on_board yes) (dnp no)
-    (property "Reference" "C8" (at 229.87 142.24 0)
-      (effects (font (size 1.27 1.27)) (justify left))
-    )
-    (property "Value" "2.2uF" (at 229.87 144.78 0)
-      (effects (font (size 1.27 1.27)) (justify left))
-    )
-    (property "Footprint" "Capacitor_THT:C_Disc_D3.0mm_W1.6mm_P2.50mm" (at 225.7552 147.32 0)
-      (effects (font (size 1.27 1.27)) hide)
-    )
-    (property "Datasheet" "~" (at 224.79 143.51 0)
-      (effects (font (size 1.27 1.27)) hide)
-    )
-    (pin "1")
-    (pin "2")
-    (instances
-      (project "DIPduino"
-        (path "/2b19a4dd-043a-4133-8ff3-f6499add1fd2"
-          (reference "C8") (unit 1)
-        )
-      )
-    )
-  )
   (symbol (lib_id "MCU_Microchip_ATmega:ATmega328P-P") (at 50.8 148.59 0) (unit 1)
     (in_bom yes) (on_board yes) (dnp no)
@@
       (effects (font (size 1.27 1.27)))
     )
-    (property "Value" "ATmega328P-PU" (at 67.31 186.69 0)
-      (effects (font (size 1.27 1.27)))
-    )
+    (property "Value" "ATMEGA328P-PU" (at 67.31 186.69 0)
+      (effects (font (size 1.27 1.27)))
+    )
