File: DIPduino.kicad_sch (KiCad schematic)
At the start: 39 parts, among them J1 USB_B, J10 3.3V Rail, J11 GND Rail, J2 BARREL JACK, J3 AVR ICSP, J4 5V Rail, J5 PIC ICSP, J6 Analog Pins, J7 Digital Pins 0-7, J8 Power Pins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

Commit message: fixed traces, improved symbol
Parts:
- C7: value 0.1uF -> 0.33uF
Connections:
- net A2: no longer U1.26 (PC3)
- net A3: now also U1.26 (PC3)
Changed lines of the file:
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@@
     (effects (font (size 1.27 1.27)) (justify left bottom))
   )
-  (label "A2" (at 66.04 148.59 0) (fields_autoplaced)
+  (label "A3" (at 66.04 148.59 0) (fields_autoplaced)
     (effects (font (size 1.27 1.27)) (justify left bottom))
   )
@@
       (effects (font (size 1.27 1.27)) (justify left))
     )
-    (property "Value" "0.1uF" (at 179.07 144.78 0)
-      (effects (font (size 1.27 1.27)) (justify left))
-    )
+    (property "Value" "0.33uF" (at 179.07 144.78 0)
+      (effects (font (size 1.27 1.27)) (justify left))
+    )
